File: dual RS232 to TTL/dual RS232 to TTL.kicad_sch (KiCad schematic)
At the start: 5 parts

Commit message: finalizado el esquema
Parts:
- added C1: 0.1uF, Capacitor_SMD:C_0402_1005Metric, symbol Herranz - Capacitor (0402):Gen_C
- added C2: 10pf, Capacitor_SMD:C_0402_1005Metric, symbol Herranz - Capacitor (0402):Gen_C
- added C3: 0.1uF, Capacitor_SMD:C_0805_2012Metric, symbol Herranz - Capacitor (0805):Gen_C
- added F1: ~, symbol Herranz - Ferrite:Gen_F
- added J1: Conn2x4, symbol Herranz - Conn Molex:Conn2x4
- added J2: Conn2x3, symbol Herranz - Conn Molex:Conn2x3
Connections:
- net +3V3: now also F1.1, J1.1 (Pin_1), J1.5 (Pin_5); no longer U?.16 (VCC)
- net GND: now also C1.2, C2.2, C3.2, J1.4 (Pin_4), J1.8 (Pin_8), J2.3 (Pin_3), J2.6 (Pin_6)
- net RX0_RS232: now also J2.5 (Pin_5)
- net RX0_TTL: now also J1.6 (Pin_6)
- net RX1_RS232: now also J2.2 (Pin_2)
- net RX1_TTL: now also J1.2 (Pin_2)
- net TX0_RS232: now also J2.4 (Pin_4)
- net TX0_TTL: now also J1.7 (Pin_7)
- net TX1_RS232: now also J2.1 (Pin_1)
- net TX1_TTL: now also J1.3 (Pin_3)
- new net: C1.1, C2.1, C3.1, F1.2, U?.16 (VCC)

Commit message: update casi finalizado
Parts:
- F1: footprint (none) -> Inductor_SMD:L_0402_1005Metric_Pad0.77x0.64mm_HandSolder
- J1: footprint (none) -> Connector_Molex:Molex_Nano-Fit_105314-xx08_2x04_P2.50mm_Horizontal
- J2: footprint (none) -> Connector_Molex:Molex_Nano-Fit_105314-xx06_2x03_P2.50mm_Horizontal
- gave numbers to parts that had none: 5
- renumbered C3 to C1, C1 to C2, C2 to C4

Commit message: PCB acabada
Parts:
- J1: footprint Connector_Molex:Molex_Nano-Fit_105314-xx08_2x04_P2.50mm_Horizontal -> Herranz - Conn Molex:Molex_Nano-Fit_105314-xx08_2x04_P2.50mm_Horizontal
- J2: footprint Connector_Molex:Molex_Nano-Fit_105314-xx06_2x03_P2.50mm_Horizontal -> Herranz - Conn Molex:Molex_Nano-Fit_105314-xx06_2x03_P2.50mm_Horizontal; MPN (none) -> 1053141106
Changed lines of the file:
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@@
   )
   (text_box "NanoFit Output fila doble:\n1 TX1 232	|4	TX0	232 |\n2 RX1 232	|5	RX0 232	|\n3 GND		|6	GND		|\n	  "
-    (at 199 122 0) (size 28 10)
+    (at 199 122 0) (size 36 14)
     (stroke (width 0) (type default))
     (fill (type none))
@@
   )
   (text_box "NanoFit Input fila doble:\n1 3v3		|5	3v3		|\n2 RX1 TTL	|6	RX0 TTL	|\n3 TX1 TTL	|7	TX0	TTL	|\n4 GND		|8	GND		|	  "
-    (at 46 105 0) (size 29 14)
+    (at 46 105 0) (size 38 18)
     (stroke (width 0) (type default))
     (fill (type none))
@@
       (effects (font (size 1.27 1.27)))
     )
-    (property "Footprint" "Connector_Molex:Molex_Nano-Fit_105314-xx06_2x03_P2.50mm_Horizontal" (at 213 104 0)
+    (property "Footprint" "Herranz - Conn Molex:Molex_Nano-Fit_105314-xx06_2x03_P2.50mm_Horizontal" (at 213 104 0)
       (effects (font (size 1.27 1.27)) hide)
     )
     (property "Datasheet" "" (at 213 104 0)
+      (effects (font (size 1.27 1.27)) hide)
+    )
+    (property "MPN" "1053141106" (at 213 104 0)
       (effects (font (size 1.27 1.27)) hide)
     )
@@
       (effects (font (size 1.27 1.27)))
     )
-    (property "Footprint" "Connector_Molex:Molex_Nano-Fit_105314-xx08_2x04_P2.50mm_Horizontal" (at 60 80 0)
-      (effects (font (size 1.27 1.27)) hide)
-    )
+    (property "Footprint" "Herranz - Conn Molex:Molex_Nano-Fit_105314-xx08_2x04_P2.50mm_Horizontal" (at 60 80 0)
+      (effects (font (size 1.27 1.27)) hide)
+    )

Commit message: Añadido agujero al PCB y Creado el archivo de producción
Parts:
- added MC1, MC2: M3_Hole, Herranz - Various:M3_Hole, symbol Herranz - Various:M3_Hole
Connections:
- net GND: now also MC1.1, MC2.1
Changed lines of the file:
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@@
+    )
+  )
+  (symbol (lib_id "power:GND") (at 60 134 0) (unit 1)
+    (in_bom yes) (on_board yes) (dnp no) (fields_autoplaced)
+    (property "Reference" "#PWR015" (at 60 140.35 0)
+      (effects (font (size 1.27 1.27)) hide)
+    )
+    (property "Value" "GND" (at 60 139.03 0)
+      (effects (font (size 1.27 1.27)))
+    )
+    (property "Footprint" "" (at 60 134 0)
+      (effects (font (size 1.27 1.27)) hide)
+    )
+    (property "Datasheet" "" (at 60 134 0)
+      (effects (font (size 1.27 1.27)) hide)
+    )
+    (pin "1")
+    (instances
+      (project "dual RS232 to TTL"
+        (path "/f83ce306-b975-4db1-ad17-124677330e47"
+          (reference "#PWR015") (unit 1)
+        )
+      )
     )
   )
@@
         (path "/f83ce306-b975-4db1-ad17-124677330e47"
           (reference "C4") (unit 1)
+        )
+      )
+    )
+  )
+  (symbol (lib_id "Herranz - Various:M3_Hole") (at 60 127 0) (unit 1)
+    (in_bom no) (on_board yes) (dnp no) (fields_autoplaced)
+    (property "Reference" "MC2" (at 63.5 131.635 0)
+      (effects (font (size 1.27 1.27)) (justify left))
+    )
+    (property "Value" "M3_Hole" (at 60 135 0)
+      (effects (font (size 1.27 1.27)) hide)
+    )
+    (property "Footprint" "Herranz - Various:M3_Hole" (at 60 127 0)
+      (effects (font (size 1.27 1.27)) hide)
+    )
+    (property "Datasheet" "" (at 60 127 0)
+      (effects (font (size 1.27 1.27)) hide)
+    )
+    (pin "1")
+    (instances
+      (project "dual RS232 to TTL"
+        (path "/f83ce306-b975-4db1-ad17-124677330e47"
+          (reference "MC2") (unit 1)
+        )
+      )
+    )
+  )
+  (symbol (lib_id "power:GND") (at 47 134 0) (unit 1)
+    (in_bom yes) (on_board yes) (dnp no) (fields_autoplaced)
+    (property "Reference" "#PWR014" (at 47 140.35 0)
+      (effects (font (size 1.27 1.27)) hide)
+    )
+    (property "Value" "GND" (at 47 139.03 0)
+      (effects (font (size 1.27 1.27)))
+    )
+    (property "Footprint" "" (at 47 134 0)
+      (effects (font (size 1.27 1.27)) hide)
+    )
+    (property "Datasheet" "" (at 47 134 0)
+      (effects (font (size 1.27 1.27)) hide)
+    )
+    (pin "1")
+    (instances
+      (project "dual RS232 to TTL"
+        (path "/f83ce306-b975-4db1-ad17-124677330e47"
+          (reference "#PWR014") (unit 1)
         )
       )
@@
         )
       )
+    )
+  )
+  (symbol (lib_id "Herranz - Various:M3_Hole") (at 47 127 0) (unit 1)
+    (in_bom no) (on_board yes) (dnp no) (fields_autoplaced)
+    (property "Reference" "MC1" (at 50.8 131.635 0)
+      (effects (font (size 1.27 1.27)) (justify left))
+    )
+    (property "Value" "M3_Hole" (at 47 135 0)
+      (effects (font (size 1.27 1.27)) hide)
+    )
+    (property "Footprint" "Herranz - Various:M3_Hole" (at 47 127 0)
+      (effects (font (size 1.27 1.27)) hide)
+    )
+    (property "Datasheet" "" (at 47 127 0)
+      (effects (font (size 1.27 1.27)) hide)
+    )
+    (pin "1")
+    (instances
+      (project "dual RS232 to TTL"
+        (path "/f83ce306-b975-4db1-ad17-124677330e47"
+          (reference "MC1") (unit 1)
+        )
+      )
